Commit message: Imported upstream version '0.1.0' of 'upstream'

File: romeo_description/urdf/romeo_generated_urdf/romeo_arms.xacro (robot description, xacro)
@@ -13,6 +13,6 @@
 	<link name="LShoulder">
 		<inertial>
-			<mass value="0.43527"/>
-			<inertia ixx="0.000268738" ixy="-7.98278e-05" ixz="8.02495e-06" iyy="0.000151197" iyz="1.72313e-05" izz="0.000290161"/>
+			<mass value="0.541429"/>
+			<inertia ixx="0.00033428" ixy="-9.92972e-05" ixz="9.98217e-06" iyy="0.000188073" iyz="2.14339e-05" izz="0.000360929"/>
 			<origin rpy="0 0 0" xyz="-0.0112798 -0.0260712 0.00468882"/>
 		</inertial>
@@ -27,6 +27,6 @@
 	<link name="LShoulderYaw_link">
 		<inertial>
-			<mass value="0.69262"/>
-			<inertia ixx="0.000953111" ixy="0.000479248" ixz="0.000898232" iyy="0.00250956" iyz="-1.65544e-05" izz="0.00233103"/>
+			<mass value="0.861545"/>
+			<inertia ixx="0.00118557" ixy="0.000596133" ixz="0.0011173" iyy="0.00312162" iyz="-2.05919e-05" izz="0.00289955"/>
 			<origin rpy="0 0 0" xyz="0.0965281 0.00465308 0.00168775"/>
 		</inertial>
@@ -42,6 +42,6 @@
 	<link name="LForeArm">
 		<inertial>
-			<mass value="0.48271"/>
-			<inertia ixx="0.000166894" ixy="9.68978e-06" ixz="-1.49781e-05" iyy="0.000408141" iyz="1.2555e-06" izz="0.00036684"/>
+			<mass value="0.600439"/>
+			<inertia ixx="0.000207598" ixy="1.2053e-05" ixz="-1.86312e-05" iyy="0.000507683" iyz="1.56171e-06" izz="0.000456309"/>
 			<origin rpy="0 0 0" xyz="-0.0348859 -0.0011589 -0.00148134"/>
 		</inertial>
@@ -56,6 +56,6 @@
 	<link name="LElbow">
 		<inertial>
-			<mass value="0.36997"/>
-			<inertia ixx="0.000404839" ixy="0.000470943" ixz="2.57237e-05" iyy="0.00102723" iyz="2.9528e-05" izz="0.000987329"/>
+			<mass value="0.460203"/>
+			<inertia ixx="0.000503576" ixy="0.000585803" ixz="3.19975e-05" iyy="0.00127777" iyz="3.67296e-05" izz="0.00122813"/>
 			<origin rpy="0 0 0" xyz="0.068523 0.0097 0.00458766"/>
 		</inertial>
@@ -71,6 +71,6 @@
 	<link name="LWristRoll_link">
 		<inertial>
-			<mass value="0.17551"/>
-			<inertia ixx="8.1046e-05" ixy="-1.46219e-06" ixz="-3.67139e-05" iyy="0.000308979" iyz="-8.92509e-08" izz="0.000294305"/>
+			<mass value="0.218316"/>
+			<inertia ixx="0.000100812" ixy="-1.81881e-06" ixz="-4.56681e-05" iyy="0.000384336" iyz="-1.11019e-07" izz="0.000366084"/>
 			<origin rpy="0 0 0" xyz="-0.0592449 6e-05 -0.00144745"/>
 		</inertial>
@@ -86,6 +86,6 @@
 	<link name="LWristYaw_link">
 		<inertial>
-			<mass value="0.061"/>
-			<inertia ixx="1.25161e-05" ixy="-4.16668e-08" ixz="-7.01768e-07" iyy="2.83374e-05" iyz="1.56375e-08" izz="2.79694e-05"/>
+			<mass value="0.0758774"/>
+			<inertia ixx="1.55687e-05" ixy="-5.1829e-08" ixz="-8.72923e-07" iyy="3.52487e-05" iyz="1.94513e-08" izz="3.4791e-05"/>
 			<origin rpy="0 0 0" xyz="-0.00657144 0.00017 -0.000115829"/>
 		</inertial>
@@ -101,6 +101,6 @@
 	<link name="l_wrist">
 		<inertial>
-			<mass value="0.35549"/>
-			<inertia ixx="0.000325271" ixy="-0.000324985" ixz="1.52493e-05" iyy="0.000666741" iyz="6.27901e-05" izz="0.000820118"/>
+			<mass value="0.442191"/>
+			<inertia ixx="0.000404603" ixy="-0.000404247" ixz="1.89685e-05" iyy="0.000829354" iyz="7.81042e-05" izz="0.00102014"/>
 			<origin rpy="0 0 0" xyz="0.07358 -0.00628 -0.00098"/>
 		</inertial>
@@ -114,5 +114,10 @@
 		<limit effort="0.649997" lower="0" upper="1.0" velocity="59.8925"/>
 	</joint>
-	<link name="l_gripper"/>
+	<link name="l_gripper">
+		<inertial>
+			<mass value="2e-06"/>
+			<inertia ixx="1.1e-09" ixy="0" ixz="0" iyy="1.1e-09" iyz="0" izz="1.1e-09"/>
+		</inertial>
+	</link>
 	<joint name="RShoulderPitch" type="revolute">
 		<parent link="torso"/>
@@ -124,6 +129,6 @@
 	<link name="RShoulder">
 		<inertial>
-			<mass value="0.43527"/>
-			<inertia ixx="0.000264235" ixy="8.24341e-05" ixz="1.55448e-05" iyy="0.000160752" iyz="-3.06968e-05" izz="0.000285109"/>
+			<mass value="0.541429"/>
+			<inertia ixx="0.00032868" ixy="0.000102539" ixz="1.9336e-05" iyy="0.000199958" iyz="-3.81835e-05" izz="0.000354645"/>
 			<origin rpy="0 0 0" xyz="-0.0112798 0.0260712 0.00468882"/>
 		</inertial>
@@ -138,6 +143,6 @@
 	<link name="RShoulderYaw_link">
 		<inertial>
-			<mass value="0.69262"/>
-			<inertia ixx="0.000955527" ixy="-0.000291705" ixz="0.000927729" iyy="0.00250758" iyz="1.49948e-05" izz="0.00233059"/>
+			<mass value="0.861545"/>
+			<inertia ixx="0.00118857" ixy="-0.00036285" ixz="0.001154" iyy="0.00311916" iyz="1.86519e-05" izz="0.002899"/>
 			<origin rpy="0 0 0" xyz="0.0965281 -0.00465308 0.00168775"/>
 		</inertial>
@@ -153,6 +158,6 @@
 	<link name="RForeArm">
 		<inertial>
-			<mass value="0.48271"/>
-			<inertia ixx="0.000166993" ixy="-6.12728e-06" ixz="-1.49476e-05" iyy="0.000408038" iyz="7.67117e-07" izz="0.000366843"/>
+			<mass value="0.600439"/>
+			<inertia ixx="0.000207722" ixy="-7.62167e-06" ixz="-1.85932e-05" iyy="0.000507556" iyz="9.54211e-07" izz="0.000456313"/>
 			<origin rpy="0 0 0" xyz="-0.0348859 0.0011589 -0.00148134"/>
 		</inertial>
@@ -167,6 +172,6 @@
 	<link name="RElbow">
 		<inertial>
-			<mass value="0.36997"/>
-			<inertia ixx="0.000404839" ixy="-2.08748e-05" ixz="2.57237e-05" iyy="0.00102723" iyz="-3.39957e-06" izz="0.000987329"/>
+			<mass value="0.460203"/>
+			<inertia ixx="0.000503576" ixy="-2.59661e-05" ixz="3.19975e-05" iyy="0.00127777" iyz="-4.2287e-06" izz="0.00122813"/>
 			<origin rpy="0 0 0" xyz="0.068523 -0.0097 0.00458766"/>
 		</inertial>
@@ -182,6 +187,6 @@
 	<link name="RWristRoll_link">
 		<inertial>
-			<mass value="0.17551"/>
-			<inertia ixx="8.1046e-05" ixy="-2.14425e-07" ixz="-3.67139e-05" iyy="0.000308979" iyz="-5.87658e-08" izz="0.000294305"/>
+			<mass value="0.218316"/>
+			<inertia ixx="0.000100812" ixy="-2.66721e-07" ixz="-4.56681e-05" iyy="0.000384336" iyz="-7.30984e-08" izz="0.000366084"/>
 			<origin rpy="0 0 0" xyz="-0.0592449 -6e-05 -0.00144745"/>
 		</inertial>
@@ -197,6 +202,6 @@
 	<link name="RWristYaw_link">
 		<inertial>
-			<mass value="0.061"/>
-			<inertia ixx="1.25161e-05" ixy="9.4625e-08" ixz="-7.01768e-07" iyy="2.83374e-05" iyz="1.80397e-08" izz="2.79694e-05"/>
+			<mass value="0.0758774"/>
+			<inertia ixx="1.55687e-05" ixy="1.17703e-07" ixz="-8.72923e-07" iyy="3.52487e-05" iyz="2.24395e-08" izz="3.4791e-05"/>
 			<origin rpy="0 0 0" xyz="-0.00657144 -0.00017 -0.000115829"/>
 		</inertial>
@@ -212,6 +217,6 @@
 	<link name="r_wrist">
 		<inertial>
-			<mass value="0.35549"/>
-			<inertia ixx="0.000325271" ixy="3.54589e-06" ixz="1.52493e-05" iyy="0.000666741" iyz="5.84145e-05" izz="0.000820118"/>
+			<mass value="0.442191"/>
+			<inertia ixx="0.000404603" ixy="4.4107e-06" ixz="1.89685e-05" iyy="0.000829354" iyz="7.26613e-05" izz="0.00102014"/>
 			<origin rpy="0 0 0" xyz="0.07358 0.00628 -0.00098"/>
 		</inertial>
@@ -225,4 +230,9 @@
 		<limit effort="0.649997" lower="0" upper="1.0" velocity="59.8925"/>
 	</joint>
-	<link name="r_gripper"/>
+	<link name="r_gripper">
+		<inertial>
+			<mass value="2e-06"/>
+			<inertia ixx="1.1e-09" ixy="0" ixz="0" iyy="1.1e-09" iyz="0" izz="1.1e-09"/>
+		</inertial>
+	</link>
 </robot>

File: romeo_description/urdf/romeo_generated_urdf/romeo_fingers.xacro (robot description, xacro)
@@ -3,6 +3,10 @@
  ****** File automatically generated by generate_urdf.py script ******
  *********************************************************************-->
-<robot name="romeoH37" xmlns:xacro="http://www.ros.org/wiki/xacro">
+<robot name="RomeoH37" xmlns:xacro="http://www.ros.org/wiki/xacro">
 	<link name="RFinger13_link">
+		<inertial>
+			<mass value="2e-06"/>
+			<inertia ixx="1.1e-09" ixy="0" ixz="0" iyy="1.1e-09" iyz="0" izz="1.1e-09"/>
+		</inertial>
 		<xacro:insert_visu_RFinger13_link/>
 	</link>
@@ -15,4 +19,8 @@
 	</joint>
 	<link name="RFinger12_link">
+		<inertial>
+			<mass value="2e-06"/>
+			<inertia ixx="1.1e-09" ixy="0" ixz="0" iyy="1.1e-09" iyz="0" izz="1.1e-09"/>
+		</inertial>
 		<xacro:insert_visu_RFinger12_link/>
 	</link>
@@ -25,4 +33,8 @@
 	</joint>
 	<link name="LFinger33_link">
+		<inertial>
+			<mass value="2e-06"/>
+			<inertia ixx="1.1e-09" ixy="0" ixz="0" iyy="1.1e-09" iyz="0" izz="1.1e-09"/>
+		</inertial>
 		<xacro:insert_visu_LFinger33_link/>
 	</link>
@@ -35,4 +47,8 @@
 	</joint>
 	<link name="RFinger31_link">
+		<inertial>
+			<mass value="2e-06"/>
+			<inertia ixx="1.1e-09" ixy="0" ixz="0" iyy="1.1e-09" iyz="0" izz="1.1e-09"/>
+		</inertial>
 		<xacro:insert_visu_RFinger31_link/>
 	</link>
@@ -45,4 +61,8 @@
 	</joint>
 	<link name="RFinger32_link">
+		<inertial>
+			<mass value="2e-06"/>
+			<inertia ixx="1.1e-09" ixy="0" ixz="0" iyy="1.1e-09" iyz="0" izz="1.1e-09"/>
+		</inertial>
 		<xacro:insert_visu_RFinger32_link/>
 	</link>
@@ -55,4 +75,8 @@
 	</joint>
 	<link name="LFinger21_link">
+		<inertial>
+			<mass value="2e-06"/>
+			<inertia ixx="1.1e-09" ixy="0" ixz="0" iyy="1.1e-09" iyz="0" izz="1.1e-09"/>
+		</inertial>
 		<xacro:insert_visu_LFinger21_link/>
 	</link>
@@ -65,4 +89,8 @@
 	</joint>
 	<link name="LFinger13_link">
+		<inertial>
+			<mass value="2e-06"/>
+			<inertia ixx="1.1e-09" ixy="0" ixz="0" iyy="1.1e-09" iyz="0" izz="1.1e-09"/>
+		</inertial>
 		<xacro:insert_visu_LFinger13_link/>
 	</link>
@@ -75,4 +103,8 @@
 	</joint>
 	<link name="LFinger32_link">
+		<inertial>
+			<mass value="2e-06"/>
+			<inertia ixx="1.1e-09" ixy="0" ixz="0" iyy="1.1e-09" iyz="0" izz="1.1e-09"/>
+		</inertial>
 		<xacro:insert_visu_LFinger32_link/>
 	</link>
@@ -85,4 +117,8 @@
 	</joint>
 	<link name="LFinger11_link">
+		<inertial>
+			<mass value="2e-06"/>
+			<inertia ixx="1.1e-09" ixy="0" ixz="0" iyy="1.1e-09" iyz="0" izz="1.1e-09"/>
+		</inertial>
 		<xacro:insert_visu_LFinger11_link/>
 	</link>
@@ -95,4 +131,8 @@
 	</joint>
 	<link name="RFinger22_link">
+		<inertial>
+			<mass value="2e-06"/>
+			<inertia ixx="1.1e-09" ixy="0" ixz="0" iyy="1.1e-09" iyz="0" izz="1.1e-09"/>
+		</inertial>
 		<xacro:insert_visu_RFinger22_link/>
 	</link>
@@ -105,4 +145,8 @@
 	</joint>
 	<link name="LFinger22_link">
+		<inertial>
+			<mass value="2e-06"/>
+			<inertia ixx="1.1e-09" ixy="0" ixz="0" iyy="1.1e-09" iyz="0" izz="1.1e-09"/>
+		</inertial>
 		<xacro:insert_visu_LFinger22_link/>
 	</link>
@@ -115,4 +159,8 @@
 	</joint>
 	<link name="RFinger21_link">
+		<inertial>
+			<mass value="2e-06"/>
+			<inertia ixx="1.1e-09" ixy="0" ixz="0" iyy="1.1e-09" iyz="0" izz="1.1e-09"/>
+		</inertial>
 		<xacro:insert_visu_RFinger21_link/>
 	</link>
@@ -125,4 +173,8 @@
 	</joint>
 	<link name="LFinger12_link">
+		<inertial>
+			<mass value="2e-06"/>
+			<inertia ixx="1.1e-09" ixy="0" ixz="0" iyy="1.1e-09" iyz="0" izz="1.1e-09"/>
+		</inertial>
 		<xacro:insert_visu_LFinger12_link/>
 	</link>
@@ -135,4 +187,8 @@
 	</joint>
 	<link name="RFinger23_link">
+		<inertial>
+			<mass value="2e-06"/>
+			<inertia ixx="1.1e-09" ixy="0" ixz="0" iyy="1.1e-09" iyz="0" izz="1.1e-09"/>
+		</inertial>
 		<xacro:insert_visu_RFinger23_link/>
 	</link>
@@ -145,4 +201,8 @@
 	</joint>
 	<link name="RFinger11_link">
+		<inertial>
+			<mass value="2e-06"/>
+			<inertia ixx="1.1e-09" ixy="0" ixz="0" iyy="1.1e-09" iyz="0" izz="1.1e-09"/>
+		</inertial>
 		<xacro:insert_visu_RFinger11_link/>
 	</link>
@@ -155,4 +215,8 @@
 	</joint>
 	<link name="LFinger23_link">
+		<inertial>
+			<mass value="2e-06"/>
+			<inertia ixx="1.1e-09" ixy="0" ixz="0" iyy="1.1e-09" iyz="0" izz="1.1e-09"/>
+		</inertial>
 		<xacro:insert_visu_LFinger23_link/>
 	</link>
@@ -165,4 +229,8 @@
 	</joint>
 	<link name="LFinger31_link">
+		<inertial>
+			<mass value="2e-06"/>
+			<inertia ixx="1.1e-09" ixy="0" ixz="0" iyy="1.1e-09" iyz="0" izz="1.1e-09"/>
+		</inertial>
 		<xacro:insert_visu_LFinger31_link/>
 	</link>
@@ -175,4 +243,8 @@
 	</joint>
 	<link name="RFinger33_link">
+		<inertial>
+			<mass value="2e-06"/>
+			<inertia ixx="1.1e-09" ixy="0" ixz="0" iyy="1.1e-09" iyz="0" izz="1.1e-09"/>
+		</inertial>
 		<xacro:insert_visu_RFinger33_link/>
 	</link>
@@ -185,4 +257,8 @@
 	</joint>
 	<link name="LThumb3_link">
+		<inertial>
+			<mass value="2e-06"/>
+			<inertia ixx="1.1e-09" ixy="0" ixz="0" iyy="1.1e-09" iyz="0" izz="1.1e-09"/>
+		</inertial>
 		<xacro:insert_visu_LThumb3_link/>
 	</link>
@@ -195,4 +271,8 @@
 	</joint>
 	<link name="LThumb1_link">
+		<inertial>
+			<mass value="2e-06"/>
+			<inertia ixx="1.1e-09" ixy="0" ixz="0" iyy="1.1e-09" iyz="0" izz="1.1e-09"/>
+		</inertial>
 		<xacro:insert_visu_LThumb1_link/>
 	</link>
@@ -205,4 +285,8 @@
 	</joint>
 	<link name="RThumb1_link">
+		<inertial>
+			<mass value="2e-06"/>
+			<inertia ixx="1.1e-09" ixy="0" ixz="0" iyy="1.1e-09" iyz="0" izz="1.1e-09"/>
+		</inertial>
 		<xacro:insert_visu_RThumb1_link/>
 	</link>
@@ -215,4 +299,8 @@
 	</joint>
 	<link name="RThumb2_link">
+		<inertial>
+			<mass value="2e-06"/>
+			<inertia ixx="1.1e-09" ixy="0" ixz="0" iyy="1.1e-09" iyz="0" izz="1.1e-09"/>
+		</inertial>
 		<xacro:insert_visu_RThumb2_link/>
 	</link>
@@ -225,4 +313,8 @@
 	</joint>
 	<link name="LThumb2_link">
+		<inertial>
+			<mass value="2e-06"/>
+			<inertia ixx="1.1e-09" ixy="0" ixz="0" iyy="1.1e-09" iyz="0" izz="1.1e-09"/>
+		</inertial>
 		<xacro:insert_visu_LThumb2_link/>
 	</link>
@@ -235,4 +327,8 @@
 	</joint>
 	<link name="RThumb3_link">
+		<inertial>
+			<mass value="2e-06"/>
+			<inertia ixx="1.1e-09" ixy="0" ixz="0" iyy="1.1e-09" iyz="0" izz="1.1e-09"/>
+		</inertial>
 		<xacro:insert_visu_RThumb3_link/>
 	</link>

File: romeo_description/urdf/romeo_generated_urdf/romeo_head.xacro (robot description, xacro)
@@ -9,10 +9,10 @@
 		<origin rpy="0 -2.98023e-08 0" xyz="0.0548 0 0.1675"/>
 		<axis xyz="0.173651 0 0.984807"/>
-		<limit effort="3.662" lower="-2.0595" upper="2.0595" velocity="4.0"/>
+		<limit effort="7.324" lower="-2.0595" upper="2.0595" velocity="4.0"/>
 	</joint>
 	<link name="NeckYaw_link">
 		<inertial>
-			<mass value="0.32745"/>
-			<inertia ixx="0.000242012" ixy="-2.69441e-07" ixz="-1.29328e-05" iyy="0.000225485" iyz="-6.99834e-07" izz="7.29248e-05"/>
+			<mass value="0.377845"/>
+			<inertia ixx="0.000279258" ixy="-3.10908e-07" ixz="-1.49231e-05" iyy="0.000260188" iyz="-8.07538e-07" izz="8.41479e-05"/>
 			<origin rpy="0 0 0" xyz="-0.00635646 0 -0.030002"/>
 		</inertial>
@@ -23,10 +23,10 @@
 		<origin rpy="0 -2.98023e-08 0" xyz="0 0 0"/>
 		<axis xyz="0 1.0 0"/>
-		<limit effort="2.978" lower="-0.3142" upper="0.6632" velocity="2.2"/>
+		<limit effort="5.956" lower="-0.3142" upper="0.6632" velocity="2.2"/>
 	</joint>
 	<link name="NeckPitch_link">
 		<inertial>
-			<mass value="0.29923"/>
-			<inertia ixx="0.000412832" ixy="-1.67846e-06" ixz="0.000111721" iyy="0.000383921" iyz="5.04259e-05" izz="0.000264006"/>
+			<mass value="0.345282"/>
+			<inertia ixx="0.000476367" ixy="-1.93678e-06" ixz="0.000128915" iyy="0.000443007" iyz="5.81865e-05" izz="0.000304636"/>
 			<origin rpy="0 0 0" xyz="0.00372 0 0.04811"/>
 		</inertial>
@@ -42,6 +42,6 @@
 	<link name="HeadPitch_link">
 		<inertial>
-			<mass value="0.13728"/>
-			<inertia ixx="2.23022e-05" ixy="1.3103e-07" ixz="-1.31933e-05" iyy="6.44652e-05" iyz="-4.26e-09" izz="5.78637e-05"/>
+			<mass value="0.158407"/>
+			<inertia ixx="2.57346e-05" ixy="1.51196e-07" ixz="-1.52238e-05" iyy="7.43865e-05" iyz="-4.91562e-09" izz="6.6769e-05"/>
 			<origin rpy="0 0 0" xyz="0.0014 0 -0.00462"/>
 		</inertial>
@@ -52,10 +52,10 @@
 		<origin rpy="0 0 0" xyz="0 0 0"/>
 		<axis xyz="1.0 0 0"/>
-		<limit effort="0.9" lower="-0.4887" upper="0.4887" velocity="1.5"/>
+		<limit effort="3.748" lower="-0.4887" upper="0.4887" velocity="1.5"/>
 	</joint>
 	<link name="HeadRoll_link">
 		<inertial>
-			<mass value="1.79432"/>
-			<inertia ixx="0.00808695" ixy="-3.36239e-05" ixz="0.00239535" iyy="0.00960886" iyz="0.000260292" izz="0.00796332"/>
+			<mass value="2.07047"/>
+			<inertia ixx="0.00933153" ixy="-3.87986e-05" ixz="0.002764" iyy="0.0110877" iyz="0.000300351" izz="0.00918888"/>
 			<origin rpy="0 0 0" xyz="0.01263 0 0.07498"/>
 		</inertial>

File: romeo_description/urdf/romeo_generated_urdf/romeo_robot.xacro (robot description, xacro)
@@ -3,5 +3,5 @@
  ****** File automatically generated by generate_urdf.py script ******
  *********************************************************************-->
-<robot name="romeoH37" xmlns:xacro="http://www.ros.org/wiki/xacro">
+<robot name="RomeoH37" xmlns:xacro="http://www.ros.org/wiki/xacro">
 	<xacro:include filename="romeo_visual_collisions.xacro"/>
 	<xacro:include filename="romeo_head.xacro"/>
@@ -12,4 +12,4 @@
 	<xacro:include filename="romeo_sensors.xacro"/>
 	<xacro:include filename="romeo_fingers.xacro"/>
-    <xacro:include filename="romeo_cap.xacro"/>
+	<xacro:include filename="romeo_cap.xacro"/>
 </robot>

File: romeo_description/urdf/romeo_generated_urdf/romeo_sensors.xacro (robot description, xacro)
@@ -3,5 +3,5 @@
  ****** File automatically generated by generate_urdf.py script ******
  *********************************************************************-->
-<robot name="romeoH37" xmlns:xacro="http://www.ros.org/wiki/xacro">
+<robot name="RomeoH37" xmlns:xacro="http://www.ros.org/wiki/xacro">
 	<link name="RFsrFToeRearRight_frame"/>
 	<joint name="RFoot/FSR/ToeRearRight_sensor_fixedjoint" type="fixed">
@@ -39,4 +39,10 @@
 		<axis xyz="0 0 0"/>
 	</joint>
+	<link name="CameraLeftEye_optical_frame"/>
+	<joint name="CameraLeftEye_optical_frame_fixedjoint" type="fixed">
+		<parent link="CameraLeftEye_frame"/>
+		<child link="CameraLeftEye_optical_frame"/>
+		<origin rpy="-1.57079632679 0 -1.57079632679" xyz="0 0 0"/>
+	</joint>
 	<link name="LFsrHeelRight_frame"/>
 	<joint name="LFoot/FSR/HeelRight_sensor_fixedjoint" type="fixed">
@@ -52,4 +58,16 @@
 		<origin rpy="0 0 0" xyz="0.01299 0 0"/>
 		<axis xyz="0 0 0"/>
+	</joint>
+	<link name="CameraRight_optical_frame"/>
+	<joint name="CameraRight_optical_frame_fixedjoint" type="fixed">
+		<parent link="CameraRight_frame"/>
+		<child link="CameraRight_optical_frame"/>
+		<origin rpy="-1.57079632679 0 -1.57079632679" xyz="0 0 0"/>
+	</joint>
+	<link name="CameraRightEye_optical_frame"/>
+	<joint name="CameraRightEye_optical_frame_fixedjoint" type="fixed">
+		<parent link="CameraRightEye_frame"/>
+		<child link="CameraRightEye_optical_frame"/>
+		<origin rpy="-1.57079632679 0 -1.57079632679" xyz="0 0 0"/>
 	</joint>
 	<link name="RFsrFToeFrontRight_frame"/>
@@ -130,4 +148,10 @@
 		<axis xyz="0 0 0"/>
 	</joint>
+	<link name="CameraLeft_optical_frame"/>
+	<joint name="CameraLeft_optical_frame_fixedjoint" type="fixed">
+		<parent link="CameraLeft_frame"/>
+		<child link="CameraLeft_optical_frame"/>
+		<origin rpy="-1.57079632679 0 -1.57079632679" xyz="0 0 0"/>
+	</joint>
 	<link name="LFsrFToeFrontRight_frame"/>
 	<joint name="LFoot/FSR/ToeFrontRight_sensor_fixedjoint" type="fixed">

File: romeo_description/urdf/romeo_generated_urdf/romeo_torso.xacro (robot description, xacro)
@@ -13,6 +13,6 @@
 	<link name="torso">
 		<inertial>
-			<mass value="5.0541"/>
-			<inertia ixx="0.0623514" ixy="-3.02711e-06" ixz="0.0093264" iyy="0.0365041" iyz="-0.000132541" izz="0.0639535"/>
+			<mass value="5.85463"/>
+			<inertia ixx="0.0587116" ixy="-3.02711e-06" ixz="0.0101426" iyy="0.0326812" iyz="-0.000132541" izz="0.0637705"/>
 			<origin rpy="0 0 0" xyz="0.01512 0 0.06743"/>
 		</inertial>
@@ -24,10 +24,10 @@
 		<origin rpy="0 0 0" xyz="0 0 0"/>
 		<axis xyz="0 0 1.0"/>
-		<limit effort="80.902" lower="-0.7575" upper="0.7575" velocity="1.5"/>
+		<limit effort="28.021" lower="-0.7575" upper="0.7575" velocity="1.5"/>
 	</joint>
 	<link name="body">
 		<inertial>
-			<mass value="4.4142"/>
-			<inertia ixx="0.0487058" ixy="6.27009e-05" ixz="-0.0496477" iyy="0.0449798" iyz="-2.92721e-05" izz="0.0182883"/>
+			<mass value="5.11337"/>
+			<inertia ixx="0.0564204" ixy="7.26322e-05" ixz="-0.0575115" iyy="0.0521042" iyz="-3.39086e-05" izz="0.021185"/>
 			<origin rpy="0 0 0" xyz="0.02825 0 -0.16653"/>
 		</inertial>
