Commit message: Imported upstream version '0.1.0' of 'upstream'

File: romeo_description/urdf/romeo_generated_urdf/romeo_visual_collisions.xacro (robot description, xacro)
@@ -4,5 +4,5 @@
  *********************************************************************-->
 <robot xmlns:xacro="http://www.ros.org/wiki/xacro">
-	<xacro:macro name="xacro:insert_visu_REye">
+	<xacro:macro name="insert_visu_REye">
 		<visual>
 			<geometry>
@@ -18,5 +18,5 @@
 		</collision>
 	</xacro:macro>
-	<xacro:macro name="xacro:insert_visu_RFinger13_link">
+	<xacro:macro name="insert_visu_RFinger13_link">
 		<visual>
 			<geometry>
@@ -32,5 +32,5 @@
 		</collision>
 	</xacro:macro>
-	<xacro:macro name="xacro:insert_visu_RThigh">
+	<xacro:macro name="insert_visu_RThigh">
 		<visual>
 			<geometry>
@@ -46,5 +46,481 @@
 		</collision>
 	</xacro:macro>
-	<xacro:macro name="xacro:insert_visu_LElbow">
+	<xacro:macro name="insert_visu_RFinger12_link">
+		<visual>
+			<geometry>
+				<mesh filename="package://romeo_description/meshes/RFinger12.dae" scale="1 1 1"/>
+			</geometry>
+			<origin rpy="0 0 0" xyz="0 0 0"/>
+		</visual>
+		<collision>
+			<geometry>
+				<mesh filename="package://romeo_description/meshes/RFinger12_0.10.stl" scale="1 1 1"/>
+			</geometry>
+			<origin rpy="0 0 0" xyz="0 0 0"/>
+		</collision>
+	</xacro:macro>
+	<xacro:macro name="insert_visu_LFinger33_link">
+		<visual>
+			<geometry>
+				<mesh filename="package://romeo_description/meshes/LFinger33.dae" scale="1 1 1"/>
+			</geometry>
+			<origin rpy="0 0 0" xyz="0 0 0"/>
+		</visual>
+		<collision>
+			<geometry>
+				<mesh filename="package://romeo_description/meshes/LFinger33_0.10.stl" scale="1 1 1"/>
+			</geometry>
+			<origin rpy="0 0 0" xyz="0 0 0"/>
+		</collision>
+	</xacro:macro>
+	<xacro:macro name="insert_visu_RFinger31_link">
+		<visual>
+			<geometry>
+				<mesh filename="package://romeo_description/meshes/RFinger31.dae" scale="1 1 1"/>
+			</geometry>
+			<origin rpy="0 0 0" xyz="0 0 0"/>
+		</visual>
+		<collision>
+			<geometry>
+				<mesh filename="package://romeo_description/meshes/RFinger31_0.10.stl" scale="1 1 1"/>
+			</geometry>
+			<origin rpy="0 0 0" xyz="0 0 0"/>
+		</collision>
+	</xacro:macro>
+	<xacro:macro name="insert_visu_LWristYaw_link">
+		<visual>
+			<geometry>
+				<mesh filename="package://romeo_description/meshes/LWristYaw.dae" scale="1 1 1"/>
+			</geometry>
+			<origin rpy="0 0 0" xyz="0 0 0"/>
+		</visual>
+		<collision>
+			<geometry>
+				<mesh filename="package://romeo_description/meshes/LWristYaw_0.10.stl" scale="1 1 1"/>
+			</geometry>
+			<origin rpy="0 0 0" xyz="0 0 0"/>
+		</collision>
+	</xacro:macro>
+	<xacro:macro name="insert_visu_RFinger32_link">
+		<visual>
+			<geometry>
+				<mesh filename="package://romeo_description/meshes/RFinger32.dae" scale="1 1 1"/>
+			</geometry>
+			<origin rpy="0 0 0" xyz="0 0 0"/>
+		</visual>
+		<collision>
+			<geometry>
+				<mesh filename="package://romeo_description/meshes/RFinger32_0.10.stl" scale="1 1 1"/>
+			</geometry>
+			<origin rpy="0 0 0" xyz="0 0 0"/>
+		</collision>
+	</xacro:macro>
+	<xacro:macro name="insert_visu_LFinger21_link">
+		<visual>
+			<geometry>
+				<mesh filename="package://romeo_description/meshes/LFinger21.dae" scale="1 1 1"/>
+			</geometry>
+			<origin rpy="0 0 0" xyz="0 0 0"/>
+		</visual>
+		<collision>
+			<geometry>
+				<mesh filename="package://romeo_description/meshes/LFinger21_0.10.stl" scale="1 1 1"/>
+			</geometry>
+			<origin rpy="0 0 0" xyz="0 0 0"/>
+		</collision>
+	</xacro:macro>
+	<xacro:macro name="insert_visu_LFinger13_link">
+		<visual>
+			<geometry>
+				<mesh filename="package://romeo_description/meshes/LFinger13.dae" scale="1 1 1"/>
+			</geometry>
+			<origin rpy="0 0 0" xyz="0 0 0"/>
+		</visual>
+		<collision>
+			<geometry>
+				<mesh filename="package://romeo_description/meshes/LFinger13_0.10.stl" scale="1 1 1"/>
+			</geometry>
+			<origin rpy="0 0 0" xyz="0 0 0"/>
+		</collision>
+	</xacro:macro>
+	<xacro:macro name="insert_visu_LFinger32_link">
+		<visual>
+			<geometry>
+				<mesh filename="package://romeo_description/meshes/LFinger32.dae" scale="1 1 1"/>
+			</geometry>
+			<origin rpy="0 0 0" xyz="0 0 0"/>
+		</visual>
+		<collision>
+			<geometry>
+				<mesh filename="package://romeo_description/meshes/LFinger32_0.10.stl" scale="1 1 1"/>
+			</geometry>
+			<origin rpy="0 0 0" xyz="0 0 0"/>
+		</collision>
+	</xacro:macro>
+	<xacro:macro name="insert_visu_LThumb3_link">
+		<visual>
+			<geometry>
+				<mesh filename="package://romeo_description/meshes/LThumb3.dae" scale="1 1 1"/>
+			</geometry>
+			<origin rpy="0 0 0" xyz="0 0 0"/>
+		</visual>
+		<collision>
+			<geometry>
+				<mesh filename="package://romeo_description/meshes/LThumb3_0.10.stl" scale="1 1 1"/>
+			</geometry>
+			<origin rpy="0 0 0" xyz="0 0 0"/>
+		</collision>
+	</xacro:macro>
+	<xacro:macro name="insert_visu_HeadRoll_link">
+		<visual>
+			<geometry>
+				<mesh filename="package://romeo_description/meshes/HeadRoll.dae" scale="1 1 1"/>
+			</geometry>
+			<origin rpy="0 0 0" xyz="0 0 0"/>
+		</visual>
+		<collision>
+			<geometry>
+				<mesh filename="package://romeo_description/meshes/HeadRoll_0.10.stl" scale="1 1 1"/>
+			</geometry>
+			<origin rpy="0 0 0" xyz="0 0 0"/>
+		</collision>
+	</xacro:macro>
+	<xacro:macro name="insert_visu_LThumb1_link">
+		<visual>
+			<geometry>
+				<mesh filename="package://romeo_description/meshes/LThumb1.dae" scale="1 1 1"/>
+			</geometry>
+			<origin rpy="0 0 0" xyz="0 0 0"/>
+		</visual>
+		<collision>
+			<geometry>
+				<mesh filename="package://romeo_description/meshes/LThumb1_0.10.stl" scale="1 1 1"/>
+			</geometry>
+			<origin rpy="0 0 0" xyz="0 0 0"/>
+		</collision>
+	</xacro:macro>
+	<xacro:macro name="insert_visu_LFinger11_link">
+		<visual>
+			<geometry>
+				<mesh filename="package://romeo_description/meshes/LFinger11.dae" scale="1 1 1"/>
+			</geometry>
+			<origin rpy="0 0 0" xyz="0 0 0"/>
+		</visual>
+		<collision>
+			<geometry>
+				<mesh filename="package://romeo_description/meshes/LFinger11_0.10.stl" scale="1 1 1"/>
+			</geometry>
+			<origin rpy="0 0 0" xyz="0 0 0"/>
+		</collision>
+	</xacro:macro>
+	<xacro:macro name="insert_visu_RFinger22_link">
+		<visual>
+			<geometry>
+				<mesh filename="package://romeo_description/meshes/RFinger22.dae" scale="1 1 1"/>
+			</geometry>
+			<origin rpy="0 0 0" xyz="0 0 0"/>
+		</visual>
+		<collision>
+			<geometry>
+				<mesh filename="package://romeo_description/meshes/RFinger22_0.10.stl" scale="1 1 1"/>
+			</geometry>
+			<origin rpy="0 0 0" xyz="0 0 0"/>
+		</collision>
+	</xacro:macro>
+	<xacro:macro name="insert_visu_LFinger22_link">
+		<visual>
+			<geometry>
+				<mesh filename="package://romeo_description/meshes/LFinger22.dae" scale="1 1 1"/>
+			</geometry>
+			<origin rpy="0 0 0" xyz="0 0 0"/>
+		</visual>
+		<collision>
+			<geometry>
+				<mesh filename="package://romeo_description/meshes/LFinger22_0.10.stl" scale="1 1 1"/>
+			</geometry>
+			<origin rpy="0 0 0" xyz="0 0 0"/>
+		</collision>
+	</xacro:macro>
+	<xacro:macro name="insert_visu_RFinger21_link">
+		<visual>
+			<geometry>
+				<mesh filename="package://romeo_description/meshes/RFinger21.dae" scale="1 1 1"/>
+			</geometry>
+			<origin rpy="0 0 0" xyz="0 0 0"/>
+		</visual>
+		<collision>
+			<geometry>
+				<mesh filename="package://romeo_description/meshes/RFinger21_0.10.stl" scale="1 1 1"/>
+			</geometry>
+			<origin rpy="0 0 0" xyz="0 0 0"/>
+		</collision>
+	</xacro:macro>
+	<xacro:macro name="insert_visu_RShoulderYaw_link">
+		<visual>
+			<geometry>
+				<mesh filename="package://romeo_description/meshes/RShoulderYaw.dae" scale="1 1 1"/>
+			</geometry>
+			<origin rpy="0 0 0" xyz="0 0 0"/>
+		</visual>
+		<collision>
+			<geometry>
+				<mesh filename="package://romeo_description/meshes/RShoulderYaw_0.10.stl" scale="1 1 1"/>
+			</geometry>
+			<origin rpy="0 0 0" xyz="0 0 0"/>
+		</collision>
+	</xacro:macro>
+	<xacro:macro name="insert_visu_LWristRoll_link">
+		<visual>
+			<geometry>
+				<mesh filename="package://romeo_description/meshes/LWristRoll.dae" scale="1 1 1"/>
+			</geometry>
+			<origin rpy="0 0 0" xyz="0 0 0"/>
+		</visual>
+		<collision>
+			<geometry>
+				<mesh filename="package://romeo_description/meshes/LWristRoll_0.10.stl" scale="1 1 1"/>
+			</geometry>
+			<origin rpy="0 0 0" xyz="0 0 0"/>
+		</collision>
+	</xacro:macro>
+	<xacro:macro name="insert_visu_RThumb1_link">
+		<visual>
+			<geometry>
+				<mesh filename="package://romeo_description/meshes/RThumb1.dae" scale="1 1 1"/>
+			</geometry>
+			<origin rpy="0 0 0" xyz="0 0 0"/>
+		</visual>
+		<collision>
+			<geometry>
+				<mesh filename="package://romeo_description/meshes/RThumb1_0.10.stl" scale="1 1 1"/>
+			</geometry>
+			<origin rpy="0 0 0" xyz="0 0 0"/>
+		</collision>
+	</xacro:macro>
+	<xacro:macro name="insert_visu_body">
+		<visual>
+			<geometry>
+				<mesh filename="package://romeo_description/meshes/TrunkYaw.dae" scale="1 1 1"/>
+			</geometry>
+			<origin rpy="0 0 0" xyz="0 0 0"/>
+		</visual>
+		<collision>
+			<geometry>
+				<mesh filename="package://romeo_description/meshes/TrunkYaw_0.10.stl" scale="1 1 1"/>
+			</geometry>
+			<origin rpy="0 0 0" xyz="0 0 0"/>
+		</collision>
+	</xacro:macro>
+	<xacro:macro name="insert_visu_RThumb2_link">
+		<visual>
+			<geometry>
+				<mesh filename="package://romeo_description/meshes/RThumb2.dae" scale="1 1 1"/>
+			</geometry>
+			<origin rpy="0 0 0" xyz="0 0 0"/>
+		</visual>
+		<collision>
+			<geometry>
+				<mesh filename="package://romeo_description/meshes/RThumb2_0.10.stl" scale="1 1 1"/>
+			</geometry>
+			<origin rpy="0 0 0" xyz="0 0 0"/>
+		</collision>
+	</xacro:macro>
+	<xacro:macro name="insert_visu_r_wrist">
+		<visual>
+			<geometry>
+				<mesh filename="package://romeo_description/meshes/RWristPitch.dae" scale="1 1 1"/>
+			</geometry>
+			<origin rpy="0 0 0" xyz="0 0 0"/>
+		</visual>
+		<collision>
+			<geometry>
+				<mesh filename="package://romeo_description/meshes/RWristPitch_0.10.stl" scale="1 1 1"/>
+			</geometry>
+			<origin rpy="0 0 0" xyz="0 0 0"/>
+		</collision>
+	</xacro:macro>
+	<xacro:macro name="insert_visu_NeckPitch_link">
+		<visual>
+			<geometry>
+				<mesh filename="package://romeo_description/meshes/NeckPitch.dae" scale="1 1 1"/>
+			</geometry>
+			<origin rpy="0 0 0" xyz="0 0 0"/>
+		</visual>
+		<collision>
+			<geometry>
+				<mesh filename="package://romeo_description/meshes/NeckPitch_0.10.stl" scale="1 1 1"/>
+			</geometry>
+			<origin rpy="0 0 0" xyz="0 0 0"/>
+		</collision>
+	</xacro:macro>
+	<xacro:macro name="insert_visu_LThumb2_link">
+		<visual>
+			<geometry>
+				<mesh filename="package://romeo_description/meshes/LThumb2.dae" scale="1 1 1"/>
+			</geometry>
+			<origin rpy="0 0 0" xyz="0 0 0"/>
+		</visual>
+		<collision>
+			<geometry>
+				<mesh filename="package://romeo_description/meshes/LThumb2_0.10.stl" scale="1 1 1"/>
+			</geometry>
+			<origin rpy="0 0 0" xyz="0 0 0"/>
+		</collision>
+	</xacro:macro>
+	<xacro:macro name="insert_visu_LFinger12_link">
+		<visual>
+			<geometry>
+				<mesh filename="package://romeo_description/meshes/LFinger12.dae" scale="1 1 1"/>
+			</geometry>
+			<origin rpy="0 0 0" xyz="0 0 0"/>
+		</visual>
+		<collision>
+			<geometry>
+				<mesh filename="package://romeo_description/meshes/LFinger12_0.10.stl" scale="1 1 1"/>
+			</geometry>
+			<origin rpy="0 0 0" xyz="0 0 0"/>
+		</collision>
+	</xacro:macro>
+	<xacro:macro name="insert_visu_RTibia">
+		<visual>
+			<geometry>
+				<mesh filename="package://romeo_description/meshes/RKneePitch.dae" scale="1 1 1"/>
+			</geometry>
+			<origin rpy="0 0 0" xyz="0 0 0"/>
+		</visual>
+		<collision>
+			<geometry>
+				<mesh filename="package://romeo_description/meshes/RKneePitch_0.10.stl" scale="1 1 1"/>
+			</geometry>
+			<origin rpy="0 0 0" xyz="0 0 0"/>
+		</collision>
+	</xacro:macro>
+	<xacro:macro name="insert_visu_LEye">
+		<visual>
+			<geometry>
+				<mesh filename="package://romeo_description/meshes/LEyePitch.dae" scale="1 1 1"/>
+			</geometry>
+			<origin rpy="0 0 0" xyz="0 0 0"/>
+		</visual>
+		<collision>
+			<geometry>
+				<mesh filename="package://romeo_description/meshes/LEyePitch_0.10.stl" scale="1 1 1"/>
+			</geometry>
+			<origin rpy="0 0 0" xyz="0 0 0"/>
+		</collision>
+	</xacro:macro>
+	<xacro:macro name="insert_visu_RWristRoll_link">
+		<visual>
+			<geometry>
+				<mesh filename="package://romeo_description/meshes/RWristRoll.dae" scale="1 1 1"/>
+			</geometry>
+			<origin rpy="0 0 0" xyz="0 0 0"/>
+		</visual>
+		<collision>
+			<geometry>
+				<mesh filename="package://romeo_description/meshes/RWristRoll_0.10.stl" scale="1 1 1"/>
+			</geometry>
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